File: Hardware/Rev. 1/Rev. 1.kicad_sch (KiCad schematic)
At the start: 1 part, among them U1 BMI160

Commit message: Initial Commit
Parts:
- removed U1: BMI160, Package_LGA:Bosch_LGA-14_3x2.5mm_P0.5mm, symbol Sensor_Motion:BMI160
- added H1: A1, symbol Mechanical:MountingHole
- added H10: D9, symbol Mechanical:MountingHole
- added H11: D10, symbol Mechanical:MountingHole
- added H12: D11, symbol Mechanical:MountingHole
- added H13: D12, symbol Mechanical:MountingHole
- added H14: VBAT, symbol Mechanical:MountingHole
- added H15, H16: NTC, symbol Mechanical:MountingHole
- added H17: VIN, symbol Mechanical:MountingHole
- added H18: VDIO, symbol Mechanical:MountingHole
- added H2: A2, symbol Mechanical:MountingHole
- added H3: A3, symbol Mechanical:MountingHole
- added H4: D0, symbol Mechanical:MountingHole
- added H5: D1, symbol Mechanical:MountingHole
- added H6: D2, symbol Mechanical:MountingHole
- added H7: D3, symbol Mechanical:MountingHole
- added H8: D7, symbol Mechanical:MountingHole
- added H9: D8, symbol Mechanical:MountingHole
- added U1: MCP4132-xxxx-P, Package_DIP:DIP-8_W7.62mm, symbol Potentiometer_Digital:MCP4132-xxxx-P
- added U2: APS6404L-3SQRx-SN, Package_SO:SOIC-8_3.9x4.9mm_P1.27mm, symbol Memory_RAM:APS6404L-3SQRx-SN
Other:
- note added: "Analog Signals"
- note added: "Digital Logic Signals"
- note added: "Memory Module"
- note added: "Mounting Holes"
- note added: "Voltage & Disconnects"
- note added: "https://docs.arduino.cc/resources/datasheets/ABX00050-datasheet.pdf"

Commit message: Started Work on Schematic
Other:
- moved on the sheet: U1
Changed lines of the file:
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@@
 	(symbol
 		(lib_id "Potentiometer_Digital:MCP4132-xxxx-P")
-		(at 143.51 90.17 0)
+		(at 152.4 86.36 0)
 		(unit 1)
 		(exclude_from_sim no)
@@
 		(fields_autoplaced yes)
 		(property "Reference" "U1"
-			(at 145.6533 77.47 0)
+			(at 154.5433 73.66 0)
 			(effects
 				(font
@@
 		)
 		(property "Value" "MCP4132-xxxx-P"
-			(at 145.6533 80.01 0)
+			(at 154.5433 76.2 0)
 			(effects
 				(font
@@
 		)
 		(property "Footprint" "Package_DIP:DIP-8_W7.62mm"
-			(at 143.51 110.49 0)
+			(at 152.4 106.68 0)
 			(effects
 				(font
@@
 		)
 		(property "Datasheet" "https://ww1.microchip.com/downloads/aemDocuments/documents/OTH/ProductDocuments/DataSheets/22060b.pdf"
-			(at 143.51 113.03 0)
+			(at 152.4 109.22 0)
 			(effects
 				(font
@@
 		)
 		(property "Description" "Single Digital Rheostat, SPI interface, 129 taps, 5/10/50/100 kohm, volatile memory"
-			(at 143.51 115.57 0)
+			(at 152.4 111.76 0)
 			(effects
 				(font

Commit message: Week 3
Parts:
- removed U1: MCP4132-xxxx-P, Package_DIP:DIP-8_W7.62mm, symbol Potentiometer_Digital:MCP4132-xxxx-P
- added BT1: LIR2032 (Rechargable), Battery:BatteryHolder_Keystone_3000_1x12mm, symbol Device:Battery
- added C1: .1 uF, Capacitor_SMD:C_0402_1005Metric, symbol Device:C
- added C2: 1 uF, Capacitor_SMD:C_0402_1005Metric, symbol Device:C
- added J1: USB_A, symbol Connector:USB_A
- added U1: TP4056-42-ESOP8, Package_SO:SOIC-8-1EP_3.9x4.9mm_P1.27mm_EP2.41x3.3mm_ThermalVias, symbol Battery_Management:TP4056-42-ESOP8
- H10, H11, H12, H13, H14, H15, H16, H17, H18: footprint (none) -> MountingHole:ToolingHole_1.152mm
Connections:
- net GND: now also U2.4 (VSS), C1.2, C2.2
- net +3.3V: now reaches U2.8 (VDD)
- net +3.3V: now also C1.1, C2.1
Other:
- note added: "Analog Inputs"
- note added: "Battery Charger (Set for 8 Hours)"
- note added: "Decoupling Capacitors"
- note added: "Digital Inputs"
- note added: "Global Labels"
- note added: "Memory Unit"
- note added: "Power Signals"
- note added: "USB Micro A (Offloading Data)"
- moved on the sheet: U2

Commit message: Week 3 Commits
Parts:
- removed BT1: LIR2032 (Rechargable), Battery:BatteryHolder_Keystone_3000_1x12mm, symbol Device:Battery
- removed H1: A1, symbol Mechanical:MountingHole
- removed H10: D9, MountingHole:ToolingHole_1.152mm, symbol Mechanical:MountingHole
- removed H11: D10, MountingHole:ToolingHole_1.152mm, symbol Mechanical:MountingHole
- removed H12: D11, MountingHole:ToolingHole_1.152mm, symbol Mechanical:MountingHole
- removed H13: D12, MountingHole:ToolingHole_1.152mm, symbol Mechanical:MountingHole
- removed H14: VBAT, MountingHole:ToolingHole_1.152mm, symbol Mechanical:MountingHole
- removed H15, H16: NTC, MountingHole:ToolingHole_1.152mm, symbol Mechanical:MountingHole
- removed H17: VIN, MountingHole:ToolingHole_1.152mm, symbol Mechanical:MountingHole
- removed H18: VDIO, MountingHole:ToolingHole_1.152mm, symbol Mechanical:MountingHole
- removed H2: A2, symbol Mechanical:MountingHole
- removed H3: A3, symbol Mechanical:MountingHole
- removed H4: D0, symbol Mechanical:MountingHole
- removed H5: D1, symbol Mechanical:MountingHole
- removed H6: D2, symbol Mechanical:MountingHole
- removed H7: D3, symbol Mechanical:MountingHole
- removed H8: D7, symbol Mechanical:MountingHole
- removed H9: D8, symbol Mechanical:MountingHole
- removed U1: TP4056-42-ESOP8, Package_SO:SOIC-8-1EP_3.9x4.9mm_P1.27mm_EP2.41x3.3mm_ThermalVias, symbol Battery_Management:TP4056-42-ESOP8
- removed U2: APS6404L-3SQRx-SN, Package_SO:SOIC-8_3.9x4.9mm_P1.27mm, symbol Memory_RAM:APS6404L-3SQRx-SN
- added BT2: CR1616, Favorites:BAT_MS621FE-FL11E, symbol Device:Battery_Cell
- added C3: 4.7 μF, Capacitor_SMD:C_0402_1005Metric, symbol Device:C
- added C4: 1 uF, Capacitor_SMD:C_0402_1005Metric, symbol Device:C
- added C5: .1 uF, Capacitor_SMD:C_0402_1005Metric, symbol Device:C
- added D1: LED_RGBK, LED_SMD:LED_Kingbright_APFA3010_3x1.5mm_Horizontal, symbol Device:LED_RGBK
- added R1: 2 kΩ, Resistor_SMD:R_0402_1005Metric, symbol Device:R_US
- added R2: 27 Ω, Resistor_SMD:R_0402_1005Metric, symbol Device:R_US
- added R3: 470 Ω, Resistor_SMD:R_0402_1005Metric, symbol Device:R_US
- added R4, R5: 10 kΩ, Resistor_SMD:R_0402_1005Metric, symbol Device:R_US
- added SW1: SW_SPST, Button_Switch_SMD:SW_DIP_SPSTx01_Slide_6.7x4.1mm_W6.73mm_P2.54mm_LowProfile_JPin, symbol Switch:SW_SPST
- added U1: MCP73831-2-OT, Package_TO_SOT_SMD:SOT-23-5, symbol Battery_Management:MCP73831-2-OT
- added U2: ~, Favorites:Arduino_Nicla_Sense_ME, symbol Favorites:Arduino_Nicla_Sense
- added U3: W25Q128JVS, Package_SO:SOIC-8_5.3x5.3mm_P1.27mm, symbol Memory_Flash:W25Q128JVS
- C1: value .1 uF -> 100 nF
- C2: value 1 uF -> 4.7 μF
- J1: footprint (none) -> Connector_USB:USB_Micro-AB_Molex_47590-0001
Connections:
- net +3.3V: now also R4.1, R5.1; no longer C1.1, C2.1
- net A1: now also U2. (4)
- net GND: now also J1.4 (GND), BT2.2 (-), C3.2, C4.2, C5.2, D1.3 (BA), R1.2, U1.2 (V_{SS}), U2. (4), U3.4 (GND)
- net VBAT: now also C4.1, C5.1, SW1.2 (B), U2. (4), U3.8 (VCC)
- net VIN: now also U2. (4)
- net at J1.1 (VBUS): now also C2.1, D1.1 (RA), U1.4 (V_{DD})
- net 3: now reaches J1.2 (D-)
- net 3: now also U2. (4)
- net 4: now reaches J1.3 (D+)
- net 4: now also U2. (4)
- net at J1.5 (Shield): now also C1.1
- new net: R3.2, U1.1 (STAT)
- new net: BT2.1 (+), C3.1, R2.2, SW1.1 (A), U1.3 (V_{BAT})
- new net: R1.1, U1.5 (PROG)
- new net: R4.2, U3.3 (~{WP}/IO_{2})
- new net: R5.2, U3.7 (~{HOLD}/~{RESET}/IO_{3})
- new net: D1.2 (GA), R2.1
- new net: D1.4 (K), R3.1
- new net 0: U2. (4)
- new net 1: U2. (4)
- new net 2: U2. (4)
- new net 5: U2. (4)
- new net 6: U2. (4), U3.1 (~{CS})
- new net 7: U2. (4), U3.5 (DI/IO_{0})
- new net 8: U2. (4), U3.2 (DO/IO_{1})
- new net 9: U2. (4), U3.6 (CLK)
- new net A0: U2. (4)
- new net VOUT: U2. (4)
Other:
- note added: "128 Mb SPI Flash Memory (~24 Hours Operation)"
- note added: "Battery Charging Circuit (Indication Lights) (500 mAh Charging)"
- note added: "Battery Protection Circuit"
- note added: "CR1616 Energizer (Rechargable Battery)"
- note added: "Memory Circuit"
- note added: "USB Micro A (Offloading Data) (Charging Battery)"
- note removed: "Analog Signals"
- note removed: "Battery Charger (Set for 8 Hours)"
- note removed: "Decoupling Capacitors"
- note removed: "Digital Logic Signals"
- note removed: "Memory Module"
- note removed: "Memory Unit"
- note removed: "Mounting Holes"
- note removed: "USB Micro A (Offloading Data)"
- note removed: "Voltage & Disconnects"
- moved on the sheet: J1

Commit message: Week 4 Changes
Parts:
- added J2: Conn_01x12_Pin, Connector_Molex:Molex_Picoflex_90325-0012_2x06_P1.27mm_Vertical, symbol Connector:Conn_01x12_Pin
Changed lines of the file:
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@@
+	)
+	(symbol
+		(lib_id "Connector:Conn_01x12_Pin")
+		(at 167.64 137.16 0)
+		(unit 1)
+		(exclude_from_sim no)
+		(in_bom yes)
+		(on_board yes)
+		(dnp no)
+		(fields_autoplaced yes)
+		(property "Reference" "J2"
+			(at 168.275 119.38 0)
+			(effects
+				(font
+					(size 1.27 1.27)
+				)
+			)
+		)
+		(property "Value" "Conn_01x12_Pin"
+			(at 168.275 121.92 0)
+			(effects
+				(font
+					(size 1.27 1.27)
+				)
+			)
+		)
+		(property "Footprint" "Connector_Molex:Molex_Picoflex_90325-0012_2x06_P1.27mm_Vertical"
+			(at 167.64 137.16 0)
+			(effects
+				(font
+					(size 1.27 1.27)
+				)
+				(hide yes)
+			)
+		)
+		(property "Datasheet" "~"
+			(at 167.64 137.16 0)
+			(effects
+				(font
+					(size 1.27 1.27)
+				)
+				(hide yes)
+			)
+		)
+		(property "Description" "Generic connector, single row, 01x12, script generated"
+			(at 167.64 137.16 0)
+			(effects
+				(font
+					(size 1.27 1.27)
+				)
+				(hide yes)
+			)
+		)
+		(pin "8"
+		)
+		(pin "10"
+		)
+		(pin "5"
+		)
+		(pin "1"
+		)
+		(pin "3"
+		)
+		(pin "2"
+		)
+		(pin "4"
+		)
+		(pin "6"
+		)
+		(pin "7"
+		)
+		(pin "9"
+		)
+		(pin "12"
+		)
+		(pin "11"
+		)
+		(instances
+			(project ""
+				(path "/2ce8eb04-2650-42ac-af18-9ab365da4f3d"
+					(reference "J2")
+					(unit 1)
+				)
+			)
+		)
 	)
 	(symbol

Commit message: Week 5 Changes
Parts:
- removed J2: Conn_01x12_Pin, Connector_Molex:Molex_Picoflex_90325-0012_2x06_P1.27mm_Vertical, symbol Connector:Conn_01x12_Pin
- removed SW1: SW_SPST, Button_Switch_SMD:SW_DIP_SPSTx01_Slide_6.7x4.1mm_W6.73mm_P2.54mm_LowProfile_JPin, symbol Switch:SW_SPST
- added C6: 1 uF, Capacitor_SMD:C_0402_1005Metric, symbol Device:C
- added C7: .1 uF, Capacitor_SMD:C_0402_1005Metric, symbol Device:C
- added D2: 1N4148WT, Diode_SMD:D_SOD-523, symbol Diode:1N4148WT
- added J2: Conn_01x12, symbol Connector_Generic:Conn_01x12
- added R6, R7: 10 kΩ, Resistor_SMD:R_0402_1005Metric, symbol Device:R_US
- added U4: W25Q32JVSS, Package_SO:SOIC-8_5.3x5.3mm_P1.27mm, symbol Memory_Flash:W25Q32JVSS
- BT2: value CR1616 -> CR2032; footprint Favorites:BAT_MS621FE-FL11E -> Battery:BatteryHolder_Keystone_1057_1x2032
Connections:
- net +3.3V: now also R6.1, R7.1
- net 0: now also U4.5 (DI/IO_{0})
- net 5: now also U4.2 (DO/IO_{1})
- net 6: now also U4.1 (~{CS})
- net 9: now also U4.6 (CLK)
- net GND: now also C6.2, C7.2, U4.4 (GND)
- net VBAT: now also C6.1, C7.1, D2.1 (K), U4.8 (VCC)
- net at BT2.1 (+), C3.1, R2.2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: now also D2.2 (A)
- new net: R6.2, U4.3 (~{WP}/IO_{2})
- new net: R7.2, U4.7 (~{HOLD}/~{RESET}/IO_{3})
Other:
- note added: "32 Mb SPI Flash Memory (~6 Hours Operation)"
- note added: "Arduino Nicla Sense + Connectors"
- note added: "Custom Symbol for Arduino Nicla Sense"
- note added: "FFC Connector (~48 pins when finished)"
- note added: "Logging for Force"
- note added: "Logging for IMU"
- note added: "Protection Diode for Battery"
- moved on the sheet: BT2, C1, C2, C3, C4, C5, D1, J1, R1, R2, R3, R4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

Commit message: Schematic Rev. 1 Finished
Parts:
- removed BT2: CR2032, Battery:BatteryHolder_Keystone_1057_1x2032, symbol Device:Battery_Cell
- removed C1: 100 nF, Capacitor_SMD:C_0402_1005Metric, symbol Device:C
- removed C6: 1 uF, Capacitor_SMD:C_0402_1005Metric, symbol Device:C
- removed C7: .1 uF, Capacitor_SMD:C_0402_1005Metric, symbol Device:C
- removed D2: 1N4148WT, Diode_SMD:D_SOD-523, symbol Diode:1N4148WT
- removed J1: USB_A, Connector_USB:USB_Micro-AB_Molex_47590-0001, symbol Connector:USB_A
- removed J2: Conn_01x12, symbol Connector_Generic:Conn_01x12
- removed R6, R7: 10 kΩ, Resistor_SMD:R_0402_1005Metric, symbol Device:R_US
- removed U2: ~, Favorites:Arduino_Nicla_Sense_ME, symbol Favorites:Arduino_Nicla_Sense
- removed U4: W25Q32JVSS, Package_SO:SOIC-8_5.3x5.3mm_P1.27mm, symbol Memory_Flash:W25Q32JVSS
- added BT1: LIR1632, footprints:BAT_504, symbol symbols:KEYSTONE_504
- added C3: 100 μF, Capacitor_SMD:C_0201_0603Metric, symbol Device:C
- added J1: 522711279, footprints:FFC_522711279, symbol symbols:522711279
- added Q1: NMOS, footprints:NMOS_DMP1045U, symbol Simulation_SPICE:NMOS
- added U2: ~, footprints:Arduino_Nicla_Sense, symbol symbols:Arduino_Nicla_Sense
- C1: renamed from C2; footprint Capacitor_SMD:C_0402_1005Metric -> Capacitor_SMD:C_0201_0603Metric
- C2: renamed from C3; footprint Capacitor_SMD:C_0402_1005Metric -> Capacitor_SMD:C_0201_0603Metric
- C4, C5: footprint Capacitor_SMD:C_0402_1005Metric -> Capacitor_SMD:C_0201_0603Metric
- R1, R2, R3, R4, R5: footprint Resistor_SMD:R_0402_1005Metric -> Resistor_SMD:R_0201_0603Metric
Connections:
- net +3.3V is gone; now on net VBAT: R4.1, R5.1
- net GND: now also BT1.N, C3.2, J1.2, J1.8, J1.P2, U2.14 (GND)
- net VBAT: now also C3.1, J1.1, J1.7, J1.P1, Q1.3 (S), U2.19 (VBAT)
- net VIN: now also C1.1, D1.1 (RA), U1.4 (V_{DD}), Q1.1 (D), U2.17 (VIN)
- net at C2.1, R2.2, U1.3 (V_{BAT}): now also BT1.P, Q1.2 (G)
- net 6 renamed 6/CS
- net 6/CS: now also U2.6 (CS)
- net 7 renamed 7/CIPO
- net 7/CIPO: now also U2.4 (CIPO)
- net 8 renamed 8/COPI
- net 8/COPI: now also U2.5 (COPI)
- net 9 renamed 9/SCLK
- net 9/SCLK: now also U2.3 (SCLK)
- new net 0/LPIO3: J1.3, J1.9, U2.13 (LPIO3)
- new net 10/A0: U2.1 (A0)
- new net 11/A1: U2.2 (A1)
- new net 1/LPIO2/RX: J1.10, J1.4, U2.12 (RX)
- new net 2/LPIO1/TX: J1.11, J1.5, U2.11 (TX)
- new net 3/SCL1: U2.10 (SCL1)
- new net 4/SDA1: U2.9 (SDA1)
- new net 5/LPIO0: J1.12, J1.6, U2.8 (LPIO0)
- new net VDDIO_EXT: U2.15 (VDDIO_EXT)
- no-connect marks 0 -> 3
Other:
- note added: "*5V Level"
- note added: "*Custom Symbol for Arduino Nicla Sense"
- note added: "*Digital Voltage Level"
- note added: "Arduino Nicla Sense ME"
- note added: "FFC Connector"
- note added: "LIR1632 (Rechargable Battery)"
- note added: "Protection MOSFET for Battery"
- note removed: "32 Mb SPI Flash Memory (~6 Hours Operation)"
- note removed: "Arduino Nicla Sense + Connectors"
- note removed: "CR1616 Energizer (Rechargable Battery)"
- note removed: "Custom Symbol for Arduino Nicla Sense"
- note removed: "FFC Connector (~48 pins when finished)"
- note removed: "Logging for Force"
- note removed: "Protection Diode for Battery"
- note removed: "USB Micro A (Offloading Data) (Charging Battery)"
- moved on the sheet: C1, C2, C4, C5, D1, R1, R2, R3, R4, R5, U1, U3

Commit message: Hardware Changes
Parts:
- removed D1: LED_RGBK, LED_SMD:LED_Kingbright_APFA3010_3x1.5mm_Horizontal, symbol Device:LED_RGBK
- removed J1: 522711279, footprints:FFC_522711279, symbol symbols:522711279
- removed R2: 27 Ω, Resistor_SMD:R_0201_0603Metric, symbol Device:R_US
- added D1: RED, Diode_SMD:D_0201_0603Metric, symbol Device:LED
- added J1: 84952-8, footprints:FFC_84952-8, symbol symbols:84952-8
- renumbered R3 to R2, R4 to R3, R5 to R4
Connections:
- net 0/LPIO3: now also J1.4
- net 10/A0: now also J1.2
- net 11/A1: now also J1.1
- net 1/LPIO2/RX: now also J1.5
- net 2/LPIO1/TX: now also J1.6
- net 5/LPIO0: now also J1.3
- net GND: now also C1.1; no longer C1.2
- net VIN: now also C1.2, D1.2 (A); no longer C1.1
- net at R2.1: now also D1.1 (K)
- new net: J1.S1 (SHIELD), J1.S2 (SHIELD)
- no-connect marks 3 -> 6
Other:
- moved on the sheet: BT1, C1, C2, C3, Q1, R1, R2, U1
