File: Hardware/Rev. 1/Rev. 1.kicad_sch (KiCad schematic)
At the start: 16 parts, among them J1 84952-8, Q1 NMOS, U1 MCP73831-2-OT, U3 W25Q128JVS

Commit message: Week 7 Changes
Parts:
- added C6: 1 uF, symbol Device:C
- added C7: 100 uF, symbol Device:C
- added C8: 10 uF, symbol Device:C
- added R10, R6, R7: 100, symbol Device:R_US
- added R5: 470, symbol Device:R_US
- added R8, R9: Rwire, symbol Device:R_US
- added U4: LM324, symbol Amplifier_Operational:LM324
Connections:
- net 3/SCL1: now also R10.1, R6.2, R7.2, R8.1
- net 4/SDA1: now also C8.2, R5.2, U4.1
- net GND: now also C6.1, C7.1, R10.2, R9.2, U4.3 (+)
- net VBAT: now also R6.1, R7.1
- new net FORCE+: C6.2, C7.2, C8.1, R5.1, U4.2 (-)
- new net STRAIN+: R8.2
- new net STRAIN-: R9.1
Other:
- note added: "*3.3 - 3.7 V"
- note added: "*Digital Voltage"
- note added: "Battery Charging Circuit"
- note added: "Charge Amplifier Circuit"
- note added: "FFC Connector Circuit"
- note added: "Force Signals"
- note added: "Red Indicator Light 500 mAh Charging"
- note added: "Strain Gauge Circuit"
- note removed: "*5V Level"
- note removed: "*Digital Voltage Level"
- note removed: "Battery Charging Circuit (Indication Lights) (500 mAh Charging)"
- note removed: "Battery Protection Circuit"
- note removed: "FFC Connector"
