File: Hardware/Rev. 1/Rev. 1.kicad_pcb (KiCad board)
At the start: 2 copper layers, 1 part

Commit message: Week 3
Parts:
- added BT1: LIR2032 (Rechargable), Battery:BatteryHolder_Keystone_3000_1x12mm, B.Cu at (171.0, 74.5)
- added U2: APS6404L-3SQRx-SN, Package_SO:SOIC-8_3.9x4.9mm_P1.27mm, F.Cu at (171.0, 79.0)
- added U2: APS6404L-3SQRx-SN, Package_SO:SOIC-8_3.9x4.9mm_P1.27mm, F.Cu at (171.0, 70.4)

Commit message: Week 3 Commits
Parts:
- removed A**: Arduino_Nicla_Vision_Socket, Favorites:Arduino_Nicla_Vision_Socket
- removed BT1: LIR2032 (Rechargable), Battery:BatteryHolder_Keystone_3000_1x12mm
- removed the U2 at (171.0, 79.0)
- removed the U2 at (171.0, 70.4)
- added BT2: CR1616, Favorites:BAT_MS621FE-FL11E, F.Cu at (171.6, 112.0)
- added C1: 100 nF, Capacitor_SMD:C_0402_1005Metric, F.Cu at (150.9, 65.0)
- added C2: 4.7 μF, Capacitor_SMD:C_0402_1005Metric, F.Cu at (150.9, 67.0)
- added C3: 4.7 μF, Capacitor_SMD:C_0402_1005Metric, F.Cu at (150.9, 68.9)
- added C4: 1 uF, Capacitor_SMD:C_0402_1005Metric, F.Cu at (150.9, 70.9)
- added C5: .1 uF, Capacitor_SMD:C_0402_1005Metric, F.Cu at (150.9, 72.9)
- added D1: LED_RGBK, LED_SMD:LED_Kingbright_APFA3010_3x1.5mm_Horizontal, F.Cu at (183.7, 94.4)
- added J1: USB_A, Connector_USB:USB_Micro-AB_Molex_47590-0001, F.Cu at (171.6, 94.0)
- added R1: 2 kΩ, Resistor_SMD:R_0402_1005Metric, F.Cu at (148.0, 65.0)
- added R2: 27 Ω, Resistor_SMD:R_0402_1005Metric, F.Cu at (148.0, 67.0)
- added R3: 470 Ω, Resistor_SMD:R_0402_1005Metric, F.Cu at (148.0, 69.0)
- added R4: 10 kΩ, Resistor_SMD:R_0402_1005Metric, F.Cu at (148.0, 71.0)
- added R5: 10 kΩ, Resistor_SMD:R_0402_1005Metric, F.Cu at (148.0, 73.0)
- added SW1: SW_SPST, Button_Switch_SMD:SW_DIP_SPSTx01_Slide_6.7x4.1mm_W6.73mm_P2.54mm_LowProfile_JPin, F.Cu at (179.6, 110.1)
- added U1: MCP73831-2-OT, Package_TO_SOT_SMD:SOT-23-5, F.Cu at (179.6, 99.7)
- added U2: ~, Favorites:Arduino_Nicla_Sense_ME, F.Cu at (164.2, 93.0)
- added U3: W25Q128JVS, Package_SO:SOIC-8_5.3x5.3mm_P1.27mm, B.Cu at (179.6, 108.2)
Routing:
- net (no net): track 0.00 -> 0.95 mm
Other:
- board outline added: 23.4 x 23.4 mm

Commit message: Week 4 Changes
Parts:
- added J2: Conn_01x12_Pin, Connector_Molex:Molex_Picoflex_90325-0012_2x06_P1.27mm_Vertical, B.Cu at (179.6, 111.6)

Commit message: Week 5 Changes
Parts:
- added D2: 1N4148WT, Diode_SMD:D_SOD-523, B.Cu at (208.6, 101.5)
- added J3: Conn_01x06_Pin, Connector_PinSocket_2.54mm:PinSocket_1x06_P2.54mm_Horizontal, B.Cu at (207.5, 105.6)
- BT2: value CR1616 -> CR2032; footprint Favorites:BAT_MS621FE-FL11E -> Battery:BatteryHolder_Keystone_1057_1x2032
- moved BT2 62.1 mm to (233.4, 106.1), turned to 0 degrees
- moved J1 57.9 mm to (221.5, 123.4), turned to 0 degrees
Other:
- board size 23.4 x 23.4 mm -> 29.4 x 23 mm

Commit message: Schematic Rev. 1 Finished
Parts:
- removed BT2: CR2032, Battery:BatteryHolder_Keystone_1057_1x2032
- removed D2: 1N4148WT, Diode_SMD:D_SOD-523
- removed the J1 at (221.5, 123.4)
- removed J2: Conn_01x12_Pin, Connector_Molex:Molex_Picoflex_90325-0012_2x06_P1.27mm_Vertical
- removed J3: Conn_01x06_Pin, Connector_PinSocket_2.54mm:PinSocket_1x06_P2.54mm_Horizontal
- removed SW1: SW_SPST, Button_Switch_SMD:SW_DIP_SPSTx01_Slide_6.7x4.1mm_W6.73mm_P2.54mm_LowProfile_JPin
- removed the U1 at (179.6, 99.7)
- removed the U2 at (164.2, 93.0)
- removed the U3 at (179.6, 108.2)
- added BT1: LIR1632, footprints:BAT_504, B.Cu at (156.1, 92.1)
- added J1: 522711279, footprints:FFC_522711279, F.Cu at (201.0, 84.5)
- added J1: 522711279, footprints:FFC_522711279, F.Cu at (160.9, 93.8)
- added Q1: NMOS, footprints:NMOS_DMP1045U, F.Cu at (155.0, 83.6)
- added U1: MCP73831-2-OT, Package_TO_SOT_SMD:SOT-23-5, F.Cu at (187.0, 81.5)
- added U1: MCP73831-2-OT, Package_TO_SOT_SMD:SOT-23-5, F.Cu at (124.6, 93.4)
- added U1: MCP73831-2-OT, Package_TO_SOT_SMD:SOT-23-5, F.Cu at (150.5, 89.2)
- added U2: ~, footprints:Arduino_Nicla_Sense, F.Cu at (180.9, 65.6)
- added U2: ~, footprints:Arduino_Nicla_Sense, F.Cu at (144.7, 80.7)
- added U3: W25Q128JVS, Package_SO:SOIC-8_5.3x5.3mm_P1.27mm, F.Cu at (150.7, 98.5)
- added U3: W25Q128JVS, Package_SO:SOIC-8_5.3x5.3mm_P1.27mm, F.Cu at (196.5, 71.2)
- C1: value 100 nF -> 4.7 μF; footprint Capacitor_SMD:C_0402_1005Metric -> Capacitor_SMD:C_0201_0603Metric
- C2, C4, C5: footprint Capacitor_SMD:C_0402_1005Metric -> Capacitor_SMD:C_0201_0603Metric
- C3: value 4.7 μF -> 100 μF; footprint Capacitor_SMD:C_0402_1005Metric -> Capacitor_SMD:C_0201_0603Metric
- R1, R2, R3, R4, R5: footprint Resistor_SMD:R_0402_1005Metric -> Resistor_SMD:R_0201_0603Metric
- moved C4 43.2 mm to (183.2, 99.4)
- moved C5 43.2 mm to (183.2, 101.4)
- moved C1 43.2 mm to (183.2, 93.5)
- moved C2 43.2 mm to (183.2, 95.5)
- moved C3 43.2 mm to (183.2, 97.5)
- moved R3 43.2 mm to (180.4, 97.5)
- moved R2 43.2 mm to (180.4, 95.5)
- moved R4 43.2 mm to (180.4, 99.5)
- moved R5 43.2 mm to (180.4, 101.5)
- moved D1 37.4 mm to (148.2, 82.4)
- moved R1 30.8 mm to (130.6, 90.5)
Connections:
- C1 pad 1: Net-(J1-Shield) -> VIN
- C2 pad 1: Net-(D1-RA) -> Net-(Q1-G)
- C3 pad 1: Net-(BT2-+) -> VBAT
- D1 pad 1: Net-(D1-RA) -> VIN
- R2 pad 2: Net-(BT2-+) -> Net-(Q1-G)
- R4 pad 1: +3.3V -> VBAT
- R5 pad 1: +3.3V -> VBAT
Routing:
- net VIN: track 0.00 -> 21.0 mm
- net GND: track 0.00 -> 1.09 mm
- net (no net): track 0.95 -> 0.00 mm
- added copper zone on F.Cu, net GND
- added copper zone on F.Cu, net VBAT
Other:
- board size 29.4 x 23 mm -> 23.4 x 23.4 mm

Commit message: Hardware Changes
Parts:
- removed the J1 at (201.0, 84.5)
- removed the J1 at (160.9, 93.8)
- removed the R2 at (180.4, 95.5)
- removed the U1 at (187.0, 81.5)
- removed the U1 at (150.5, 89.2)
- removed the U2 at (180.9, 65.6)
- removed the U3 at (196.5, 71.2)
- added J1: 84952-8, footprints:FFC_84952-8, F.Cu at (179.5, 77.8)
- D1: value LED_RGBK -> RED; footprint LED_SMD:LED_Kingbright_APFA3010_3x1.5mm_Horizontal -> Diode_SMD:D_0201_0603Metric
- moved D1 47.4 mm to (185.1, 112.1)
- moved U3 36.1 mm to (173.6, 70.5), turned to -90 degrees
- moved U2 29.0 mm to (168.1, 63.6)
- renumbered R3 to R2, R4 to R3, R5 to R4
Connections:
- C1 pad 1: VIN -> GND
- C1 pad 2: GND -> VIN
- D1 pad 1: VIN -> Net-(D1-K)
- D1 pad 2: Net-(D1-GA) -> VIN
Routing:
- net VIN: track 21.0 -> 0.00 mm
- net 10/A0: track 0.00 -> 13.5 mm
- net 5/LPIO0: track 0.00 -> 12.6 mm
- net 0/LPIO3: track 0.00 -> 12.2 mm
- net 1/LPIO2/RX: track 0.00 -> 11.9 mm
- net 11/A1: track 0.00 -> 11.8 mm
- net 2/LPIO1/TX: track 0.00 -> 11.6 mm
- net GND: track 1.09 -> 0.00 mm
Other:
- copper layers 2 -> 4

Commit message: Week 7 Changes
Parts:
- moved R1 57.8 mm to (183.1, 66.3)
- moved U1 57.8 mm to (177.1, 69.3)
- moved BT1 19.8 mm to (147.4, 74.3)
- moved U3 10.5 mm to (183.8, 73.2), turned to 0 degrees
- moved J1 0.66 mm to (179.0, 78.2)
Changed lines of the file:
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@@
 	(footprint "Resistor_SMD:R_0201_0603Metric"
 		(layer "F.Cu")
-		(at 130.58 90.45)
+		(at 183.08 66.35)
 		(descr "Resistor SMD 0201 (0603 Metric), square (rectangular) end terminal, IPC-7351 nominal, (Body size source: https://www.vishay.com/docs/20052/crcw0201e3.pdf), generated with kicad-footprint-generator")
 		(tags "resistor")
@@
 	(footprint "footprints:FFC_84952-8"
 		(layer "F.Cu")
-		(at 179.5 77.8)
+		(at 179 78.225)
 		(property "Reference" "J1"
 			(at -4.825 -2.385 0)
@@
 	(footprint "Package_SO:SOIC-8_5.3x5.3mm_P1.27mm"
 		(layer "F.Cu")
-		(at 173.6 70.55 -90)
+		(at 183.7875 73.21)
 		(descr "SOIC, 8 Pin (JEITA/EIAJ ED-7311-19 variation 08-001-BBA and Atmel/Microchip, 208 mils width, https://www.jeita.or.jp/japanese/standard/book/ED-7311-19/#target/page_no=21, https://ww1.microchip.com/downloads/en/DeviceDoc/20005045C.pdf#page=23, https://ww1.microchip.com/downloads/en/DeviceDoc/doc2535.pdf#page=162), generated with kicad-footprint-generator ipc_gullwing_generator.py")
 		(tags "SOIC SO P-SOP SOP SOP-8 SO SO-8 8S2 S2AE/F K04-056 CASE-751BE SO8W 8-Pin-SOIC PSA W8-2 W8-4 W8MS-1 FPT-8P-M08")
 		(property "Reference" "U3"
-			(at 0 -3.6 90)
+			(at 0 -3.6 0)
 			(layer "F.SilkS")
 			(hide yes)
@@
 		)
 		(property "Value" "W25Q128JVS"
-			(at 0 3.6 90)
+			(at 0 3.6 0)
 			(layer "F.Fab")
 			(hide yes)
@@
 		)
 		(property "Datasheet" "https://www.winbond.com/resource-files/w25q128jv_dtr%20revc%2003272018%20plus.pdf"
-			(at 0 0 90)
+			(at 0 0 0)
 			(layer "F.Fab")
 			(hide yes)
@@
 		)
 		(property "Description" "128Mbit / 16MiB Serial Flash Memory, Standard/Dual/Quad SPI, 2.7-3.6V, SOIC-8"
-			(at 0 0 90)
+			(at 0 0 0)
 			(layer "F.Fab")
 			(hide yes)
@@
 		(attr smd)
 		(fp_line
-			(start -2.76 2.76)
-			(end -2.76 2.49)
+			(start -2.76 -2.76)
+			(end -2.76 -2.49)
 			(stroke
 				(width 0.12)
@@
 		)
 		(fp_line
-			(start 0 2.76)
-			(end -2.76 2.76)
+			(start -2.76 2.76)
+			(end -2.76 2.49)
 			(stroke
 				(width 0.12)
@@
 		)
 		(fp_line
-			(start 0 2.76)
-			(end 2.76 2.76)
+			(start 0 -2.76)
+			(end -2.76 -2.76)
 			(stroke
 				(width 0.12)
@@
 		)
 		(fp_line
-			(start 2.76 2.76)
-			(end 2.76 2.49)
+			(start 0 -2.76)
+			(end 2.76 -2.76)
 			(stroke
 				(width 0.12)
@@
 		)
 		(fp_line
-			(start -2.76 -2.76)
-			(end -2.76 -2.49)
+			(start 0 2.76)
+			(end -2.76 2.76)
 			(stroke
 				(width 0.12)
@@
 		)
 		(fp_line
-			(start 0 -2.76)
-			(end -2.76 -2.76)
+			(start 0 2.76)
+			(end 2.76 2.76)
 			(stroke
 				(width 0.12)
@@
 		)
 		(fp_line
-			(start 0 -2.76)
-			(end 2.76 -2.76)
+			(start 2.76 -2.76)
+			(end 2.76 -2.49)
 			(stroke
 				(width 0.12)
@@
 		)
 		(fp_line
-			(start 2.76 -2.76)
-			(end 2.76 -2.49)
+			(start 2.76 2.76)
+			(end 2.76 2.49)
 			(stroke
 				(width 0.12)
@@
 		)
 		(fp_line
-			(start -2.9 2.9)
-			(end -2.9 2.48)
+			(start -4.65 -2.48)
+			(end -2.9 -2.48)
 			(stroke
 				(width 0.05)
@@
 		)
 		(fp_line
-			(start 2.9 2.9)
-			(end -2.9 2.9)
+			(start -4.65 2.48)
+			(end -4.65 -2.48)
 			(stroke
 				(width 0.05)
@@
 		)
 		(fp_line
-			(start -4.65 2.48)
-			(end -4.65 -2.48)
+			(start -2.9 -2.9)
+			(end 2.9 -2.9)
 			(stroke
 				(width 0.05)
@@
 		)
 		(fp_line
-			(start -2.9 2.48)
-			(end -4.65 2.48)
+			(start -2.9 -2.48)
+			(end -2.9 -2.9)
 			(stroke
 				(width 0.05)
@@
 		)
 		(fp_line
-			(start 2.9 2.48)
-			(end 2.9 2.9)
+			(start -2.9 2.48)
+			(end -4.65 2.48)
 			(stroke
 				(width 0.05)
@@
 		)
 		(fp_line
-			(start 4.65 2.48)
-			(end 2.9 2.48)
+			(start -2.9 2.9)
+			(end -2.9 2.48)
 			(stroke
 				(width 0.05)
@@
 		)
 		(fp_line
-			(start -4.65 -2.48)
-			(end -2.9 -2.48)
+			(start 2.9 -2.9)
+			(end 2.9 -2.48)
 			(stroke
 				(width 0.05)
@@
 		)
 		(fp_line
-			(start -2.9 -2.48)
-			(end -2.9 -2.9)
+			(start 2.9 -2.48)
+			(end 4.65 -2.48)
 			(stroke
 				(width 0.05)
@@
 		)
 		(fp_line
-			(start 2.9 -2.48)
-			(end 4.65 -2.48)
+			(start 2.9 2.48)
+			(end 2.9 2.9)
 			(stroke
 				(width 0.05)
@@
 		)
 		(fp_line
-			(start 4.65 -2.48)
-			(end 4.65 2.48)
+			(start 2.9 2.9)
+			(end -2.9 2.9)
 			(stroke
 				(width 0.05)
@@
 		)
 		(fp_line
-			(start -2.9 -2.9)
-			(end 2.9 -2.9)
+			(start 4.65 -2.48)
+			(end 4.65 2.48)
 			(stroke
 				(width 0.05)
@@
 		)
 		(fp_line
-			(start 2.9 -2.9)
-			(end 2.9 -2.48)
+			(start 4.65 2.48)
+			(end 2.9 2.48)
 			(stroke
 				(width 0.05)
@@
 		)
 		(fp_text user "${REFERENCE}"
-			(at 0 0 90)
+			(at 0 0 0)
 			(layer "F.Fab")
 			(effects
@@
 		)
 		(pad "1" smd roundrect
-			(at -3.5875 -1.905 270)
+			(at -3.5875 -1.905)
 			(size 1.625 0.65)
 			(layers "F.Cu" "F.Mask" "F.Paste")
@@
 		)
 		(pad "2" smd roundrect
-			(at -3.5875 -0.635 270)
+			(at -3.5875 -0.635)
 			(size 1.625 0.65)
 			(layers "F.Cu" "F.Mask" "F.Paste")
@@
 		)
 		(pad "3" smd roundrect
-			(at -3.5875 0.635 270)
+			(at -3.5875 0.635)
 			(size 1.625 0.65)
 			(layers "F.Cu" "F.Mask" "F.Paste")
@@
 		)
 		(pad "4" smd roundrect
-			(at -3.5875 1.905 270)
+			(at -3.5875 1.905)
 			(size 1.625 0.65)
 			(layers "F.Cu" "F.Mask" "F.Paste")
@@
 		)
 		(pad "5" smd roundrect
-			(at 3.5875 1.905 270)
+			(at 3.5875 1.905)
 			(size 1.625 0.65)
 			(layers "F.Cu" "F.Mask" "F.Paste")
@@
 		)
 		(pad "6" smd roundrect
-			(at 3.5875 0.635 270)
+			(at 3.5875 0.635)
 			(size 1.625 0.65)
 			(layers "F.Cu" "F.Mask" "F.Paste")
@@
 		)
 		(pad "7" smd roundrect
-			(at 3.5875 -0.635 270)
+			(at 3.5875 -0.635)
 			(size 1.625 0.65)
 			(layers "F.Cu" "F.Mask" "F.Paste")
@@
 		)
 		(pad "8" smd roundrect
-			(at 3.5875 -1.905 270)
+			(at 3.5875 -1.905)
 			(size 1.625 0.65)
 			(layers "F.Cu" "F.Mask" "F.Paste")
@@
 	(footprint "Package_TO_SOT_SMD:SOT-23-5"
 		(layer "F.Cu")
-		(at 124.575 93.4375)
+		(at 177.075 69.3375)
 		(descr "SOT, 5 Pin (JEDEC MO-178 Var AA https://www.jedec.org/document_search?search_api_views_fulltext=MO-178), generated with kicad-footprint-generator ipc_gullwing_generator.py")
 		(tags "SOT TO_SOT_SMD")
@@
 	(footprint "footprints:BAT_504"
 		(layer "B.Cu")
-		(at 156.085 92.105 -90)
+		(at 147.375 74.275 -90)
 		(property "Reference" "BT1"
 			(at -11.415 9.885 90)
@@
 		(polygon
 			(pts
-				(xy 124.075 94.075) (xy 118.6 94.075) (xy 118.525 97.825) (xy 123.975 97.85) (xy 124.125 97.85)
-				(xy 124.175 94.075) (xy 124.175 94.05)
+				(xy 176.575 69.975) (xy 171.1 69.975) (xy 171.025 73.725) (xy 176.475 73.75) (xy 176.625 73.75)
+				(xy 176.675 69.975) (xy 176.675 69.95)
 			)
 		)
@@
 		(min_thickness 0.25)
 		(filled_areas_thickness no)
-		(fill
+		(fill yes
 			(thermal_gap 0.5)
 			(thermal_bridge_width 0.5)
@@
 		(polygon
 			(pts
-				(xy 124.15 93.75) (xy 121.825 93.75) (xy 121.825 93.125) (xy 118.65 93.075) (xy 118.65 89.575) (xy 122.525 89.625)
-				(xy 122.525 92.175) (xy 126.625 92.2) (xy 126.625 90.525) (xy 133.125 90.45) (xy 133.125 92.7) (xy 128.425 92.7)
-				(xy 128.425 93.725)
+				(xy 176.65 69.65) (xy 174.325 69.65) (xy 174.325 69.025) (xy 171.15 68.975) (xy 171.15 65.475) (xy 175.025 65.525)
+				(xy 175.025 68.075) (xy 179.125 68.1) (xy 179.125 66.425) (xy 185.625 66.35) (xy 185.625 68.6) (xy 180.925 68.6)
+				(xy 180.925 69.625)
 			)
 		)
