File: Hardware/Rev. 3/Rev. 3.kicad_pcb (KiCad board)
At the start: 4 copper layers, 23.4 x 23.4 mm, 16 parts, among them J1 84952-8, Q1 NMOS, U1 MCP73831-2-OT, U3 W25Q128JVS

Commit message: Week 12 Changes
Parts:
- removed C3: 100 μF, Capacitor_SMD:C_0201_0603Metric
- removed C5: .1 uF, Capacitor_SMD:C_0201_0603Metric
- removed J1: 84952-8, footprints:FFC_84952-8
- removed Q1: NMOS, footprints:NMOS_DMP1045U
- added D2: 1N4148WT, Diode_SMD:D_SOD-523, F.Cu at (223.0, 71.8)
- BT1: value LIR1632 -> LIR2032
- R1: value 2 kΩ -> 2.2 kΩ
- moved BT1 72.6 mm to (219.2, 85.3)
- moved D1 45.1 mm to (215.4, 78.7), turned to 180 degrees
- moved C2 42.0 mm to (219.9, 74.9), turned to -90 degrees
- moved R2 41.4 mm to (217.0, 78.2), turned to 90 degrees
- moved U2 40.9 mm to (207.6, 74.2)
- moved U1 39.9 mm to (216.5, 75.4), turned to 180 degrees
- moved R4 38.3 mm to (214.2, 83.6)
- moved R3 35.5 mm to (212.1, 83.6), turned to 180 degrees
- moved U3 35.3 mm to (215.5, 88.7), turned to 90 degrees
- moved C1 35.1 mm to (213.0, 74.9), turned to 90 degrees
- moved R1 34.3 mm to (215.4, 77.8), turned to 180 degrees
- moved C4 31.0 mm to (210.6, 84.7), turned to 90 degrees
Connections:
- net Net-(Q1-G) renamed DIODE
Routing:
- net GND: track 0.00 -> 44.3 mm, vias 0 -> 3
- net VBAT: track 0.00 -> 28.6 mm, vias 0 -> 2
- net VIN: track 0.00 -> 21.9 mm
- net Net-(U3-~{WP}/IO_{2}): track 0.00 -> 17.2 mm, vias 0 -> 2
- net 10/A0: track 13.5 -> 0.00 mm
- net 5/LPIO0: track 12.6 -> 0.00 mm
- net 0/LPIO3: track 12.2 -> 0.00 mm
- net 1/LPIO2/RX: track 11.9 -> 0.00 mm
- net 11/A1: track 11.8 -> 0.00 mm
- net 2/LPIO1/TX: track 11.6 -> 0.00 mm
- net 9/SCLK: track 0.00 -> 10.6 mm
- net 7/CIPO: track 0.00 -> 9.52 mm
- net 8/COPI: track 0.00 -> 7.78 mm
- net 6/CS: track 0.00 -> 5.33 mm
- net Net-(U1-STAT): track 0.00 -> 1.85 mm
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- added copper zone on B.Cu, net DIODE
- added copper zone on F.Cu, net DIODE
- added copper zone on B.Cu, net GND
- added copper zone on B.Cu, net VIN
- added copper zone on F.Cu, net VIN
- removed copper zone on F.Cu, net VBAT
Other:
- board size 23.4 x 23.4 mm -> 25.5 x 32.7 mm
