File: Hardware/Rev. 3/Rev. 3.kicad_sch (KiCad schematic)
At the start: 26 parts, among them J1 84952-8, Q1 NMOS, U1 MCP73831-2-OT, U3 W25Q128JVS, U4 LM324

Commit message: Week 12 Changes
Parts:
- removed C3: 100 μF, Capacitor_SMD:C_0201_0603Metric, symbol Device:C
- removed C5: .1 uF, Capacitor_SMD:C_0201_0603Metric, symbol Device:C
- removed C6: 1 uF, symbol Device:C
- removed C7: 100 uF, symbol Device:C
- removed C8: 10 uF, symbol Device:C
- removed J1: 84952-8, footprints:FFC_84952-8, symbol symbols:84952-8
- removed Q1: NMOS, footprints:NMOS_DMP1045U, symbol Simulation_SPICE:NMOS
- removed R10, R6, R7: 100, symbol Device:R_US
- removed R5: 470, symbol Device:R_US
- removed R8, R9: Rwire, symbol Device:R_US
- removed U4: LM324, symbol Amplifier_Operational:LM324
- added D2: 1N4148WT, Diode_SMD:D_SOD-523, symbol Diode:1N4148WT
- BT1: value LIR1632 -> LIR2032
- R1: value 2 kΩ -> 2.2 kΩ
Connections:
- net VBAT: now also D2.2 (A)
- net at BT1.P, C2.1, U1.3 (V_{BAT}): now also D2.1 (K)
- no-connect marks 6 -> 3
Other:
- note added: ".1 uF Denoising capacitor removed to save space"
- note added: "Charge Protection is already included in the MCP73831 IC"
- note added: "LIR2032 (Rechargable Battery)"
- note removed: "Charge Amplifier Circuit"
- note removed: "FFC Connector Circuit"
- note removed: "Force Signals"
- note removed: "LIR1632 (Rechargable Battery)"
- note removed: "Protection MOSFET for Battery"
- note removed: "Strain Gauge Circuit"
- title: Nathan Huang Board Design -> Keel Bone PCB (Data Storage and Battery Only)
- moved on the sheet: C1, C4, R2, R3, U3

Commit message: Week 12 Changes
Connections:
- net DIODE: now reaches BT1.P, C2.1, D2.1 (K), U1.3 (V_{BAT})
Changed lines of the file:
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@@
+		)
+	)
+	(global_label "DIODE"
+		(shape input)
+		(at 97.79 53.34 90)
+		(fields_autoplaced yes)
+		(effects
+			(font
+				(size 1.27 1.27)
+			)
+			(justify left)
+		)
+		(property "Intersheetrefs" "${INTERSHEET_REFS}"
+			(at 97.79 44.7305 90)
+			(effects
+				(font
+					(size 1.27 1.27)
+				)
+				(justify left)
+				(hide yes)
+			)
 		)
 	)

Commit message: Week 3
Parts:
- C1, C2, C4: footprint Capacitor_SMD:C_0201_0603Metric -> Capacitor_SMD:C_0504_1310Metric_Pad0.83x1.28mm_HandSolder
- D1: footprint Diode_SMD:D_0201_0603Metric -> Diode_SMD:D_0603_1608Metric_Pad1.05x0.95mm_HandSolder
- R1, R2, R3, R4: footprint Resistor_SMD:R_0201_0603Metric -> Resistor_SMD:R_0402_1005Metric_Pad0.72x0.64mm_HandSolder
Changed lines of the file:
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@@
 			)
 		)
-		(property "Footprint" "Diode_SMD:D_0201_0603Metric"
+		(property "Footprint" "Diode_SMD:D_0603_1608Metric_Pad1.05x0.95mm_HandSolder"
 			(at 60.96 39.37 0)
 			(effects
@@
 			)
 		)
-		(property "Footprint" "Capacitor_SMD:C_0201_0603Metric"
+		(property "Footprint" "Capacitor_SMD:C_0504_1310Metric_Pad0.83x1.28mm_HandSolder"
 			(at 30.7848 40.64 0)
 			(effects
@@
 			)
 		)
-		(property "Footprint" "Resistor_SMD:R_0201_0603Metric"
+		(property "Footprint" "Resistor_SMD:R_0402_1005Metric_Pad0.72x0.64mm_HandSolder"
 			(at 28.194 136.144 90)
 			(effects
@@
 			)
 		)
-		(property "Footprint" "Resistor_SMD:R_0201_0603Metric"
+		(property "Footprint" "Resistor_SMD:R_0402_1005Metric_Pad0.72x0.64mm_HandSolder"
 			(at 42.164 68.834 90)
 			(effects
@@
 			)
 		)
-		(property "Footprint" "Resistor_SMD:R_0201_0603Metric"
+		(property "Footprint" "Resistor_SMD:R_0402_1005Metric_Pad0.72x0.64mm_HandSolder"
 			(at 28.194 125.984 90)
 			(effects
@@
 			)
 		)
-		(property "Footprint" "Resistor_SMD:R_0201_0603Metric"
+		(property "Footprint" "Resistor_SMD:R_0402_1005Metric_Pad0.72x0.64mm_HandSolder"
 			(at 72.136 47.244 90)
 			(effects
@@
 			)
 		)
-		(property "Footprint" "Capacitor_SMD:C_0201_0603Metric"
+		(property "Footprint" "Capacitor_SMD:C_0504_1310Metric_Pad0.83x1.28mm_HandSolder"
 			(at 79.7052 60.96 0)
 			(effects
@@
 			)
 		)
-		(property "Footprint" "Capacitor_SMD:C_0201_0603Metric"
+		(property "Footprint" "Capacitor_SMD:C_0504_1310Metric_Pad0.83x1.28mm_HandSolder"
 			(at 89.8652 128.27 0)
 			(effects

Commit message: Changes
Parts:
- C1, C2, C4: footprint Capacitor_SMD:C_0504_1310Metric_Pad0.83x1.28mm_HandSolder -> Capacitor_SMD:C_0402_1005Metric_Pad0.74x0.62mm_HandSolder
Changed lines of the file:
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@@
 			)
 		)
-		(property "Footprint" "Capacitor_SMD:C_0504_1310Metric_Pad0.83x1.28mm_HandSolder"
+		(property "Footprint" "Capacitor_SMD:C_0402_1005Metric_Pad0.74x0.62mm_HandSolder"
 			(at 30.7848 40.64 0)
 			(effects
@@
 			)
 		)
-		(property "Footprint" "Capacitor_SMD:C_0504_1310Metric_Pad0.83x1.28mm_HandSolder"
+		(property "Footprint" "Capacitor_SMD:C_0402_1005Metric_Pad0.74x0.62mm_HandSolder"
 			(at 79.7052 60.96 0)
 			(effects
@@
 			)
 		)
-		(property "Footprint" "Capacitor_SMD:C_0504_1310Metric_Pad0.83x1.28mm_HandSolder"
+		(property "Footprint" "Capacitor_SMD:C_0402_1005Metric_Pad0.74x0.62mm_HandSolder"
 			(at 89.8652 128.27 0)
 			(effects
