File: Hardware/Rev. 4/Rev.4.kicad_pcb (KiCad board)
At the start: 4 copper layers, 25.5 x 32.7 mm, 24 parts, among them U1 MCP73831-2-OT, U3 W25Q128JVS, U5 PCC110

Commit message: Week 17 Changes
Parts:
- removed AE1: Antenna, RF_Antenna:NiceRF_SW868-TH13_868Mhz
- removed C6: 1 uF, Capacitor_SMD:C_0201_0603Metric
- removed C7: 100 uF, Capacitor_SMD:C_0201_0603Metric
- removed C8: 10 uF, Capacitor_SMD:C_0201_0603Metric
- removed R5: 470, Resistor_SMD:R_0201_0603Metric
- removed U5: PCC110, Package_TO_SOT_SMD:TO-252-3_TabPin2
- added C3: 1 uF, Capacitor_SMD:C_0201_0603Metric, F.Cu at (216.1, 100.8)
- added C5: 100 uF, Capacitor_SMD:C_0201_0603Metric, F.Cu at (217.1, 100.9)
- added U4: AD7150, footprints:AD7150, F.Cu at (214.9, 96.3)
- R10, R6, R7: value 100 -> 1 kΩ
- R8, R9: value Rwire -> 1.5 kΩ
- moved R6 7.70 mm to (226.2, 89.2)
- moved R7 4.07 mm to (226.3, 86.7)
- moved R9 2.98 mm to (226.3, 79.1), turned to 180 degrees
- moved R8 1.61 mm to (225.7, 81.9), turned to 180 degrees
- moved R10 0.61 mm to (226.3, 84.2)
Connections:
- net FORCE- renamed GND
- R10 pad 1: 3/SCL1 -> 0/LPIO3
- R6 pad 2: 3/SCL1 -> 0/LPIO3
- R7 pad 2: 3/SCL1 -> 0/LPIO3
- R8 pad 1: 3/SCL1 -> 0/LPIO3
Routing:
- net 3/SCL1: track 0.00 -> 26.8 mm
- net VBAT: track 28.6 -> 48.6 mm
- net 4/SDA1: track 0.00 -> 17.5 mm
- net 0/LPIO3: track 0.00 -> 10.3 mm
- net GND: track 44.3 -> 52.7 mm
- added copper zone on B.Cu, net (none)
- added copper zone on F.Cu, net (none)
- removed copper zone on B.Cu, net GND
- removed copper zone on F.Cu, net GND
