File: Hardware/Rev. 4/Rev.4.kicad_sch (KiCad schematic)
At the start: 25 parts, among them U1 MCP73831-2-OT, U3 W25Q128JVS, U4 LM324, U5 PCC110

Commit message: Week 17 Changes
Parts:
- removed AE1: Antenna, RF_Antenna:NiceRF_SW868-TH13_868Mhz, symbol Device:Antenna
- removed C6: 1 uF, Capacitor_SMD:C_0201_0603Metric, symbol Device:C
- removed C7: 100 uF, Capacitor_SMD:C_0201_0603Metric, symbol Device:C
- removed C8: 10 uF, Capacitor_SMD:C_0201_0603Metric, symbol Device:C
- removed R5: 470, Resistor_SMD:R_0201_0603Metric, symbol Device:R_US
- removed U4: LM324, Converter_ACDC:Converter_ACDC_CUI_PBO-3-Sxx_THT_Vertical, symbol Amplifier_Operational:LM324
- removed U5: PCC110, Package_TO_SOT_SMD:TO-252-3_TabPin2, symbol Regulator_Linear:LM1117DT-1.8
- added C3: 1 uF, Capacitor_SMD:C_0201_0603Metric, symbol Device:C
- added C5: 100 uF, Capacitor_SMD:C_0201_0603Metric, symbol Device:C
- added U4: AD7150, footprints:AD7150, symbol symbols:AD7150
- R10, R6, R7: value 100 -> 1 kΩ
- R8, R9: value Rwire -> 1.5 kΩ
Connections:
- net 0/LPIO3: now also R10.1, R6.2, R7.2, R8.1
- net 3/SCL1: now also U4.9 (SCL); no longer R10.1, R6.2, R7.2, R8.1
- net 4/SDA1: now also U4.10 (SDA)
- net 5/LPIO0: now also U4.7 (OUT1)
- net FORCE+: now also U4.3 (CIN2)
- net GND: now also C3.2, C5.2
- net VBAT: now also U4.2 (VDD)
- new net: C3.1, C5.1, U4.1 (GND)
- new net FORCE-: U4.4 (CIN1)
- no-connect marks 3 -> 6
Other:
- note removed: "RF Charging Circuit"
- moved on the sheet: R10, R6, R7, R8, R9
