File: Hardware/Rev. 4/Rev.4.kicad_sch (KiCad schematic)
At the start: 21 parts, among them U1 MCP73831-2-OT, U3 W25Q128JVS, U4 AD7150

Commit message: Changes
Parts:
- added AE1: RFID Antenna, symbol Device:Antenna
- added P1110B: U1, symbol symbols:P1110b
- added R5: 50, symbol Device:R_US
Connections:
- net 10/A0: now also P1110B.9 (Dout)
- net GND: now also P1110B.10 (ALK), P1110B.7 (GND)
- net VIN: now also P1110B.8 (Vout)
- new net: P1110B.3 (RFin), R5.1
- new net: AE1.1 (A), R5.2
- new net RF_GND: P1110B.2 (GND), P1110B.4 (GND)
- no-connect marks 6 -> 9
Other:
- note added: "*10/A0 Pin used to read signal strength level*"
- note added: "*ALK set to DC GND to set voltage level to 3.3 V*"
- note added: "*Custom Symbol for P1110b Powercast Harvester*"
- note added: "Powercast P1110B: RFID -> DC Converter"
- moved on the sheet: C3, C5, R10, R6, R7, R8, R9, U4
