File: Hardware/Rev. 5/_autosave-Rev. 5.kicad_pcb (KiCad board)
At the start: 4 copper layers, 29.2 x 29.2 mm, 28 parts, among them J1 Conn_01x03_Pin, J2 FFC_4_Pin, U1 MCP73831-2-OT, U3 W25Q128JVS, U4 AD7150, U5 PCC110

Commit message: Week 10 Changes
Parts:
- moved U4 12.1 mm to (214.3, 88.2), turned to 90 degrees
- moved J2 6.71 mm to (222.7, 96.0)
- moved U3 4.14 mm to (222.4, 87.7)
- moved J1 0.66 mm to (213.4, 97.2), turned to 180 degrees
