File: Hardware/Rev. 6/Rev. 6.kicad_pcb (KiCad board)
At the start: 2 copper layers, 45 x 35 mm, 24 parts, among them J1 Conn_01x03_Pin, J2 FFC_4_Pin, U1 MCP73831-2-OT, U3 W25Q128JVS, U4 AD7150

Commit message: Changes
Parts:
- moved BT1 1.01 mm to (234.6, 85.1)
Other:
- board size 45 x 35 mm -> 42 x 34 mm
Changed lines of the file:
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@@
 	(footprint "footprints:BAT_504"
 		(layer "B.Cu")
-		(at 235.6 84.95 -90)
+		(at 234.6 85.12 -90)
 		(property "Reference" "BT1"
 			(at -11.415 9.885 90)
@@
 		)
 	)
-	(gr_arc
-		(start 238.75 67.1)
-		(mid 242.285534 68.564466)
-		(end 243.75 72.1)
+	(gr_line
+		(start 198.45 96.6)
+		(end 198.45 72.6)
 		(stroke
-			(width 0.2)
+			(width 0.05)
 			(type default)
 		)
 		(layer "Edge.Cuts")
 	)
-	(gr_line
-		(start 198.75 97.1)
-		(end 198.75 72.1)
+	(gr_arc
+		(start 198.45 72.6)
+		(mid 199.914466 69.064466)
+		(end 203.45 67.6)
 		(stroke
-			(width 0.2)
+			(width 0.05)
 			(type default)
 		)
 		(layer "Edge.Cuts")
 	)
-	(gr_arc
-		(start 243.75 97.1)
-		(mid 242.285534 100.635534)
-		(end 238.75 102.1)
+	(gr_line
+		(start 235.45 101.6)
+		(end 203.45 101.6)
 		(stroke
-			(width 0.2)
+			(width 0.05)
 			(type default)
 		)
 		(layer "Edge.Cuts")
 	)
-	(gr_line
-		(start 203.75 67.1)
-		(end 238.75 67.1)
+	(gr_arc
+		(start 240.45 96.6)
+		(mid 238.985534 100.135534)
+		(end 235.45 101.6)
 		(stroke
-			(width 0.2)
+			(width 0.05)
 			(type default)
 		)
@@
 	)
 	(gr_line
-		(start 243.75 72.1)
-		(end 243.75 97.1)
+		(start 240.45 72.6)
+		(end 240.45 96.6)
 		(stroke
-			(width 0.2)
+			(width 0.05)
 			(type default)
 		)
@@
 	)
 	(gr_arc
-		(start 198.75 72.1)
-		(mid 200.214466 68.564466)
-		(end 203.75 67.1)
+		(start 203.45 101.6)
+		(mid 199.914466 100.135534)
+		(end 198.45 96.6)
 		(stroke
-			(width 0.2)
+			(width 0.05)
 			(type default)
 		)
 		(layer "Edge.Cuts")
 	)
-	(gr_arc
-		(start 203.75 102.1)
-		(mid 200.214466 100.635534)
-		(end 198.75 97.1)
+	(gr_line
+		(start 203.45 67.6)
+		(end 235.45 67.6)
 		(stroke
-			(width 0.2)
+			(width 0.05)
 			(type default)
 		)
 		(layer "Edge.Cuts")
 	)
-	(gr_line
-		(start 238.75 102.1)
-		(end 203.75 102.1)
+	(gr_arc
+		(start 235.45 67.6)
+		(mid 238.985534 69.064466)
+		(end 240.45 72.6)
 		(stroke
-			(width 0.2)
+			(width 0.05)
 			(type default)
 		)

Commit message: Changes
Parts:
- added REF**: P1110b, footprints:P1110b, F.Cu at (233.7, 85.0)
Changed lines of the file:
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@@
 	(net 34 "unconnected-(J2-PadP1)")
 	(net 35 "unconnected-(J2-PadP2)")
+	(footprint "footprints:P1110b"
+		(layer "F.Cu")
+		(at 233.65 85 90)
+		(property "Reference" "REF**"
+			(at 0 -0.5 90)
+			(unlocked yes)
+			(layer "F.SilkS")
+			(effects
+				(font
+					(size 1 1)
+					(thickness 0.1)
+				)
+			)
+		)
+		(property "Value" "P1110b"
+			(at 0 1 90)
+			(unlocked yes)
+			(layer "F.Fab")
+			(effects
+				(font
+					(size 1 1)
+					(thickness 0.15)
+				)
+			)
+		)
+		(property "Datasheet" ""
+			(at 0 0 90)
+			(unlocked yes)
+			(layer "F.Fab")
+			(hide yes)
+			(effects
+				(font
+					(size 1 1)
+					(thickness 0.15)
+				)
+			)
+		)
+		(property "Description" ""
+			(at 0 0 90)
+			(unlocked yes)
+			(layer "F.Fab")
+			(hide yes)
+			(effects
+				(font
+					(size 1 1)
+					(thickness 0.15)
+				)
+			)
+		)
+		(attr smd)
+		(fp_line
+			(start -4.985 -5.46)
+			(end 4.985 -5.46)
+			(stroke
+				(width 0.1)
+				(type default)
+			)
+			(layer "F.SilkS")
+		)
+		(fp_line
+			(start 6.985 -3.46)
+			(end 6.985 3.46)
+			(stroke
+				(width 0.1)
+				(type default)
+			)
+			(layer "F.SilkS")
+		)
+		(fp_line
+			(start -6.985 3.46)
+			(end -6.985 -3.46)
+			(stroke
+				(width 0.1)
+				(type default)
+			)
+			(layer "F.SilkS")
+		)
+		(fp_line
+			(start 4.985 5.46)
+			(end -4.985 5.46)
+			(stroke
+				(width 0.1)
+				(type default)
+			)
+			(layer "F.SilkS")
+		)
+		(fp_arc
+			(start 4.985 -5.46)
+			(mid 6.399214 -4.874214)
+			(end 6.985 -3.46)
+			(stroke
+				(width 0.1)
+				(type default)
+			)
+			(layer "F.SilkS")
+		)
+		(fp_arc
+			(start -6.985 -3.46)
+			(mid -6.399214 -4.874214)
+			(end -4.985 -5.46)
+			(stroke
+				(width 0.1)
+				(type default)
+			)
+			(layer "F.SilkS")
+		)
+		(fp_arc
+			(start 6.985 3.46)
+			(mid 6.399214 4.874214)
+			(end 4.985 5.46)
+			(stroke
+				(width 0.1)
+				(type default)
+			)
+			(layer "F.SilkS")
+		)
+		(fp_arc
+			(start -4.985 5.46)
+			(mid -6.399214 4.874214)
+			(end -6.985 3.46)
+			(stroke
+				(width 0.1)
+				(type default)
+			)
+			(layer "F.SilkS")
+		)
+		(pad "" thru_hole circle
+			(at -4.5 -4.5 90)
+			(size 1 1)
+			(drill 0.5)
+			(layers "*.Cu" "*.Mask")
+			(remove_unused_layers no)
+		)
+		(pad "" thru_hole circle
+			(at -4.5 4.5 90)
+			(size 1 1)
+			(drill 0.5)
+			(layers "*.Cu" "*.Mask")
+			(remove_unused_layers no)
+		)
+		(pad "" thru_hole circle
+			(at 4.5 -4.5 90)
+			(size 1 1)
+			(drill 0.5)
+			(layers "*.Cu" "*.Mask")
+			(remove_unused_layers no)
+		)
+		(pad "" thru_hole circle
+			(at 4.5 4.5 90)
+			(size 1 1)
+			(drill 0.5)
+			(layers "*.Cu" "*.Mask")
+			(remove_unused_layers no)
+		)
+		(pad "1" smd roundrect
+			(at -6 -3 90)
+			(size 1.905 1.27)
+			(layers "F.Cu" "F.Mask" "F.Paste")
+			(roundrect_rratio 0.15)
+		)
+		(pad "2" smd roundrect
+			(at -6 -1.5 90)
+			(size 1.905 1.27)
+			(layers "F.Cu" "F.Mask" "F.Paste")
+			(roundrect_rratio 0.15)
+		)
+		(pad "3" smd roundrect
+			(at -6 0 90)
+			(size 1.905 1.27)
+			(layers "F.Cu" "F.Mask" "F.Paste")
+			(roundrect_rratio 0.15)
+		)
+		(pad "4" smd roundrect
+			(at -6 1.5 90)
+			(size 1.905 1.27)
+			(layers "F.Cu" "F.Mask" "F.Paste")
+			(roundrect_rratio 0.15)
+		)
+		(pad "5" smd roundrect
+			(at -6 3 90)
+			(size 1.905 1.27)
+			(layers "F.Cu" "F.Mask" "F.Paste")
+			(roundrect_rratio 0.15)
+		)
+		(pad "6" smd roundrect
+			(at 6 3 90)
+			(size 1.905 1.27)
+			(layers "F.Cu" "F.Mask" "F.Paste")
+			(roundrect_rratio 0.15)
+		)
+		(pad "7" smd roundrect
+			(at 6 1.5 90)
+			(size 1.905 1.27)
+			(layers "F.Cu" "F.Mask" "F.Paste")
+			(roundrect_rratio 0.15)
+		)
+		(pad "8" smd roundrect
+			(at 6 0 90)
+			(size 1.905 1.27)
+			(layers "F.Cu" "F.Mask" "F.Paste")
+			(roundrect_rratio 0.15)
+		)
+		(pad "9" smd roundrect
+			(at 6 -1.5 90)
+			(size 1.905 1.27)
+			(layers "F.Cu" "F.Mask" "F.Paste")
+			(roundrect_rratio 0.15)
+		)
+		(pad "10" smd roundrect
+			(at 6 -3 90)
+			(size 1.905 1.27)
+			(layers "F.Cu" "F.Mask" "F.Paste")
+			(roundrect_rratio 0.15)
+		)
+		(embedded_fonts no)
+	)
 	(footprint "Resistor_SMD:R_0805_2012Metric_Pad1.20x1.40mm_HandSolder"
 		(layer "B.Cu")

Commit message: Week 8 Changes
Parts:
- moved BT1 2.38 mm to (232.2, 85.0)
- moved REF** 1.43 mm to (232.2, 85.0)
- moved R3 1.35 mm to (222.8, 96.8)
- moved R10 1.33 mm to (222.9, 91.9)
- moved R6 1.33 mm to (222.9, 86.9)
- moved R12 1.32 mm to (222.8, 77.7)
- moved R9 1.31 mm to (222.8, 82.3)
Routing:
- net VBAT: track 0.00 -> 64.4 mm
- net 0/LPIO3: track 0.00 -> 47.5 mm, vias 0 -> 1
- net GND: track 0.00 -> 34.1 mm
- net 10/A0: track 0.00 -> 33.7 mm, vias 0 -> 1
- net 5/LPIO0: track 0.00 -> 29.4 mm, vias 0 -> 1
- net 4/SDA1: track 0.00 -> 28.4 mm, vias 0 -> 1
- net 3/SCL1: track 0.00 -> 27.2 mm, vias 0 -> 1
- net Net-(U4-GND): track 0.00 -> 21.6 mm, vias 0 -> 2
- net 9/SCLK: track 0.00 -> 21.4 mm, vias 0 -> 1
- net 7/CIPO: track 0.00 -> 20.2 mm, vias 0 -> 1
- net STRAIN+: track 0.00 -> 17.3 mm
- net 8/COPI: track 0.00 -> 13.1 mm, vias 0 -> 1
- net Net-(U3-~{HOLD}/~{RESET}/IO_{3}): track 0.00 -> 3.04 mm
- net Net-(U3-~{WP}/IO_{2}): track 0.00 -> 2.96 mm
